Commit message: Enable to move static base

File: urdf/inc/static_base.xacro (robot description, xacro)
@@ -2,9 +2,9 @@
 <robot name="static_base" xmlns:xacro="http://ros.org/wiki/xacro">
 <xacro:macro name="static_base" params="prefix arm_prefix">
-<joint name="${prefix}world_joint" type="fixed">
+<!-- <joint name="${prefix}world_joint" type="fixed">
   <parent link="world" />
   <child link = "${prefix}platform" />
   <origin xyz="0.0 0.0 0.43" rpy="0.0 0.0 0.0" />
-</joint>
+</joint> -->
 <link name='${prefix}platform'>
   <pose>0 0 0 0 0 0</pose>
@@ -17,10 +17,10 @@
   <visual>
     <geometry>
-      <box size="0.1 0.1 0.82" />
+      <box size="0.3 0.3 0.3" />
     </geometry>
   </visual>
   <collision>
     <geometry>
-      <box size="0.1 0.1 0.82" />
+      <box size="0.3 0.3 0.3" />
     </geometry>
   </collision>
@@ -29,5 +29,5 @@
   <parent link="${prefix}platform" />
   <child link = "${prefix}base_link" />
-  <origin xyz="0.0 0.0 0.43" rpy="0.0 0.0 0.0" />
+  <origin xyz="0.0 0.0 0.15" rpy="0.0 0.0 0.0" />
 </joint>
 <xacro:if value="${arm_prefix != prefix}">

File: urdf/ur_with_cam.xacro (robot description, xacro)
@@ -86,6 +86,8 @@
     />
   </xacro:if>
-  <link name='world' />
   <xacro:property name="base" value="$(arg base)"/>
+  <xacro:if value="${base != 'static'}">
+    <link name='world' />
+  </xacro:if>
   <xacro:if value="${base == 'static'}">
     <xacro:include filename="$(find ur_with_cam_gazebo)/urdf/inc/static_base.xacro"/>
@@ -119,8 +121,16 @@
     />
   </xacro:if>
-  <xacro:property name="include_room" value="$(arg include_room)"/>
+  <xacro:if value="${base == 'box'}">
+    <xacro:include filename="$(find ur_with_cam_gazebo)/urdf/inc/box.xacro"/>
+    <xacro:trollomatic
+      prefix=""
+      arm_prefix="arm_"
+      transmission_hw_interface="$(arg transmission_hw_interface)"
+    />
+  </xacro:if>
+  <!-- <xacro:property name="include_room" value="$(arg include_room)"/>
   <xacro:if value="${include_room}">
     <xacro:include filename="$(find ur_with_cam_gazebo)/urdf/inc/room.xacro"/>
     <xacro:room/>
-  </xacro:if>
+  </xacro:if> -->
 </robot>
